Commit message: feat: add dual-arm MIDI piano playback

File: src/ros2_rm_robot/rm_description/urdf/rm_75_6fb_v_dual.urdf.xacro (robot description, xacro)
@@ -6,4 +6,11 @@
   <xacro:arg name="right_rpy" default="3.14159265 1.5707963 -1.5707963" />
   <link name="base_root" />
+  <!-- Keyboard calibration frame. Key coordinates in rm_piano_player are expressed here. -->
+  <link name="piano_frame" />
+  <joint name="piano_frame_fixed" type="fixed">
+    <origin xyz="0 0 0" rpy="0 0 0" />
+    <parent link="base_root" />
+    <child link="piano_frame" />
+  </joint>
   <xacro:macro name="rm75_arm" params="prefix">
     <link name="${prefix}_base_link">

Commit message: feat: add tabletop piano scene and root guide

File: src/ros2_rm_robot/rm_description/urdf/rm_75_6fb_v_dual.urdf.xacro (robot description, xacro)
@@ -5,9 +5,10 @@
   <xacro:arg name="right_xyz" default="0 0.075 0.5" />
   <xacro:arg name="right_rpy" default="3.14159265 1.5707963 -1.5707963" />
+  <xacro:arg name="piano_xyz" default="0 0 0" />
   <link name="base_root" />
   <!-- Keyboard calibration frame. Key coordinates in rm_piano_player are expressed here. -->
   <link name="piano_frame" />
   <joint name="piano_frame_fixed" type="fixed">
-    <origin xyz="0 0 0" rpy="0 0 0" />
+    <origin xyz="$(arg piano_xyz)" rpy="0 0 0" />
     <parent link="base_root" />
     <child link="piano_frame" />

File: src/ros2_rm_robot/rm_mujoco/config/rm_75_6fb_v_dual_l20_mujoco_control.urdf.xacro (robot description, xacro)
@@ -2,15 +2,20 @@
 <robot xmlns:xacro="http://www.ros.org/wiki/xacro" name="rm_75_6fb_v_dual_l20_mujoco_control">
   <xacro:arg name="headless" default="false" />
+  <xacro:arg name="mujoco_model" default="$(find rm_mujoco)/models/rm_75_6fb_v_dual_l20.xml" />
+  <xacro:arg name="scene_config" default="$(find rm_mujoco)/config/piano_scene.yaml" />
+  <xacro:property name="initial_positions" value="${xacro.load_yaml('$(arg scene_config)')['initial_positions']}" />
   <ros2_control name="MujocoSystem" type="system">
     <hardware>
       <plugin>mujoco_ros2_control/MujocoSystemInterface</plugin>
-      <param name="mujoco_model">$(find rm_mujoco)/models/rm_75_6fb_v_dual_l20.xml</param>
+      <param name="mujoco_model">$(arg mujoco_model)</param>
       <param name="sim_speed_factor">1.0</param>
       <param name="headless">$(arg headless)</param>
+      <!-- Overview cameras are for the viewer, not ROS image streams. -->
+      <param name="auto_register_cameras">false</param>
     </hardware>
     <xacro:macro name="position_joint" params="joint_name">
       <joint name="${joint_name}">
         <command_interface name="position" />
-        <state_interface name="position"><param name="initial_value">0.0</param></state_interface>
+        <state_interface name="position"><param name="initial_value">${initial_positions.get(joint_name, 0.0)}</param></state_interface>
         <state_interface name="velocity" />
       </joint>
@@ -24,4 +29,8 @@
       <xacro:position_joint joint_name="${prefix}_joint6" />
       <xacro:position_joint joint_name="${prefix}_joint7" />
+      <joint name="${prefix}_camera_rojoint">
+        <state_interface name="position"><param name="initial_value">0.0</param></state_interface>
+        <state_interface name="velocity" />
+      </joint>
     </xacro:macro>
     <xacro:macro name="hand_joints" params="prefix">
